File: PCB/atti.kicad_pcb (KiCad board)
At the start: 2 copper layers, 109.2 x 71.1 mm, 35 parts, among them J1 Conn_02x04_Counter_Clockwise, J2 FTSH-105-01-X-D-007-K, J3 Conn_01x01_Female, J5 Conn_01x01_Female, J6 Conn_01x01_Female, J7 Conn_01x01_Female, SW1 SW_SPST, U1 AP2112K-3.3, U2 STM32F303K8Tx, U3 NVT2006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

Commit message: Second routing attempt
Parts:
- moved C2 44.3 mm to (102.3, 83.7), turned to 270 degrees
- moved U1 37.8 mm to (105.4, 83.8), turned to 270 degrees
- moved J2 36.8 mm to (109.5, 91.7), turned to 90 degrees
- moved J5 36.8 mm to (124.0, 65.5)
- moved J7 36.6 mm to (117.3, 65.5)
- moved C3 36.3 mm to (104.6, 87.4), turned to 0 degrees
- moved J1 33.3 mm to (121.7, 90.7), turned to 270 degrees
- moved J6 31.3 mm to (114.0, 65.5)
- moved R1 30.4 mm to (110.7, 66.0)
- moved J3 29.5 mm to (120.7, 65.5)
- moved R2 28.7 mm to (104.4, 67.3), turned to 0 degrees
- moved D2 27.2 mm to (104.4, 65.3), turned to 0 degrees
- moved D1 26.4 mm to (108.0, 65.3), turned to 180 degrees
- moved U6 20.2 mm to (110.0, 82.0), turned to 90 degrees
- moved C13 19.9 mm to (117.6, 84.8)
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Connections:
- J1 pad 2: Net-(J1-Pad2) -> GND
- J1 pad 8: GND -> Net-(J1-Pad8)
- U2 pad 18: BMX_INT1 -> Net-(J3-Pad1)
- U2 pad 27: Net-(J3-Pad1) -> BMX_INT1
- U3 pad 10: USART1_RTS_DE -> I2C1_SCL
- U3 pad 11: I2C1_SCL -> USART1_RTS_DE
- U3 pad 12: I2C1_SDA -> USART1_CTS
- U3 pad 13: USART1_CTS -> USART1_RX
- U3 pad 3: Net-(J1-Pad7) -> Net-(J1-Pad8)
- U3 pad 4: Net-(J1-Pad6) -> Net-(J1-Pad7)
- U3 pad 5: Net-(J1-Pad5) -> Net-(J1-Pad6)
- U3 pad 6: Net-(J1-Pad4) -> Net-(J1-Pad5)
- U3 pad 7: Net-(J1-Pad3) -> Net-(J1-Pad4)
- U3 pad 8: Net-(J1-Pad2) -> Net-(J1-Pad3)
- U3 pad 9: USART1_RX -> I2C1_SDA
Routing:
- net VDD: track 103.3 -> 49.1 mm, vias 6 -> 2
- net VIN: track 21.9 -> 52.1 mm, vias 1 -> 2
- net BMP_CSB: track 27.3 -> 0.00 mm, vias 2 -> 0
- net Net-(J1-Pad8): track 0.00 -> 22.8 mm
- net GND: track 118.7 -> 98.1 mm, vias 2 -> 3
- net SPI1_SCK: track 29.4 -> 10.4 mm, vias 2 -> 0
- net I2C1_SCL: track 3.22 -> 19.7 mm
- net Net-(J1-Pad7): track 4.88 -> 19.5 mm
- net Net-(J1-Pad6): track 7.96 -> 21.5 mm
- net I2C1_SDA: track 6.69 -> 20.0 mm, vias 1 -> 0
- net Net-(J1-Pad5): track 5.25 -> 18.3 mm
- net Net-(J1-Pad4): track 8.47 -> 21.0 mm
- net Net-(J1-Pad2): track 11.3 -> 0.00 mm
- net Net-(J1-Pad3): track 5.79 -> 16.6 mm
- net SPI1_MOSI: track 25.9 -> 15.5 mm, vias 2 -> 3
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Other:
- board size 109.2 x 71.1 mm -> 30.2 x 32 mm

Commit message: Good routing progress
Parts:
- removed J3, J5, J6, J7: Conn_01x01_Female, Connector_Wire:SolderWire-0.25sqmm_1x01_D0.65mm_OD1.7mm
- moved C6 56.8 mm to (152.7, 102.4), turned to 270 degrees
- moved C9 55.9 mm to (151.9, 96.0), turned to 180 degrees
- moved Y1 53.0 mm to (150.6, 98.8), turned to 0 degrees
- moved C10 51.2 mm to (148.3, 96.0), turned to 0 degrees
- moved R4 49.6 mm to (150.9, 115.3), turned to 180 degrees
- moved R3 48.5 mm to (147.3, 98.8), turned to 270 degrees
- moved D2 48.0 mm to (140.1, 97.3)
- moved U3 47.5 mm to (146.1, 115.3)
- moved D1 46.8 mm to (140.1, 99.3), turned to 0 degrees
- moved U2 46.3 mm to (146.3, 105.9), turned to 270 degrees
- moved R6 45.8 mm to (150.9, 113.0), turned to 0 degrees
- moved C7 44.2 mm to (144.5, 97.3), turned to 180 degrees
- moved R2 43.9 mm to (136.5, 97.3)
- moved C3 43.7 mm to (137.2, 116.6)
- moved C2 43.6 mm to (134.4, 113.3)
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Connections:
- J1 pad 1: VIN -> Net-(J1-Pad1)
- J1 pad 2: GND -> Net-(J1-Pad2)
- J1 pad 7: Net-(J1-Pad7) -> VIN
- J1 pad 8: Net-(J1-Pad8) -> GND
- U2 pad 10: Net-(J7-Pad1) -> BMX_INT2
- U2 pad 27: BMX_INT1 -> Net-(U2-Pad27)
- U2 pad 28: BMX_INT2 -> Net-(U2-Pad28)
- U2 pad 9: Net-(J6-Pad1) -> BMX_INT1
- U3 pad 3: Net-(J1-Pad8) -> Net-(J1-Pad6)
- U3 pad 4: Net-(J1-Pad7) -> Net-(J1-Pad5)
- U3 pad 5: Net-(J1-Pad6) -> Net-(J1-Pad4)
- U3 pad 6: Net-(J1-Pad5) -> Net-(J1-Pad3)
- U3 pad 7: Net-(J1-Pad4) -> Net-(J1-Pad2)
- U3 pad 8: Net-(J1-Pad3) -> Net-(J1-Pad1)
Routing:
- net VIN: track 52.1 -> 9.90 mm, vias 2 -> 0
- net GND: track 98.1 -> 72.1 mm, vias 3 -> 0
- net Net-(J1-Pad8): track 22.8 -> 0.00 mm
- net VDD: track 49.1 -> 28.7 mm, vias 2 -> 0
- net Net-(J1-Pad7): track 19.5 -> 0.00 mm
- net Net-(J1-Pad5): track 18.3 -> 3.22 mm
- net Net-(J1-Pad4): track 21.0 -> 5.95 mm
- net Net-(J1-Pad6): track 21.5 -> 6.74 mm
- net I2C1_SCL: track 19.7 -> 5.83 mm
- net Net-(J1-Pad3): track 16.6 -> 2.74 mm
- net I2C1_SDA: track 20.0 -> 6.18 mm
- net BMX_INT2: track 0.00 -> 11.8 mm, vias 0 -> 2
- net Net-(R5-Pad2): track 9.80 -> 0.77 mm, vias 2 -> 0
- net USART1_RTS_DE: track 11.2 -> 2.56 mm
- net USART1_CTS: track 9.86 -> 2.50 mm
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Other:
- board size 30.2 x 32 mm -> 27.9 x 33.3 mm

Commit message: Routing complete
Parts:
- moved R4 2.40 mm to (152.1, 113.3), turned to 270 degrees
- moved C12 2.01 mm to (133.0, 99.7)
- moved C14 2.01 mm to (133.0, 103.3)
- moved R6 1.05 mm to (149.9, 113.3), turned to 90 degrees
- moved J1 0.25 mm to (149.6, 121.2)
- moved U3 0.07 mm to (146.1, 115.4)
Routing:
- net GND: track 72.1 -> 167.9 mm, vias 0 -> 6
- net VDD: track 28.7 -> 111.0 mm, vias 0 -> 3
- net NRST: track 0.00 -> 35.7 mm, vias 0 -> 2
- net SWCLK: track 0.00 -> 29.3 mm, vias 0 -> 1
- net SWDIO: track 0.00 -> 26.6 mm, vias 0 -> 1
- net SWO: track 0.00 -> 25.0 mm, vias 0 -> 1
- net JTDI: track 0.00 -> 22.8 mm, vias 0 -> 1
- net VIN: track 9.90 -> 20.8 mm, vias 0 -> 1
- net Net-(D1-Pad2): track 0.00 -> 7.95 mm, vias 0 -> 2
- net I2C1_SDA: track 6.18 -> 13.1 mm
- net Net-(D2-Pad2): track 0.00 -> 6.95 mm
- net I2C1_SCL: track 5.83 -> 12.6 mm
- net Net-(R5-Pad2): track 0.77 -> 2.35 mm
- net BMX_INT1: track 7.31 -> 8.84 mm
